Commit message: 修复 EC616 平行夹爪安装与开合，并恢复关节限位。
源 URDF 在 gripper_1 后 XML 损坏，两指 STL 又近似相同而非镜像件，只能重建安装；过程中先后踩过装进法兰内侧、错误镜像面（含与屏幕重合的 XZ）、同号开合导致对开失败等问题，最终定为法兰 YZ 镜像（两指 ±X、铰链 +Y）并对 gripper_2 取反驱动。顺带放宽臂关节 limit，并在 URDF 回调即结束 loading，避免卡在 99%。

File: ec616/ec616.urdf (robot description, URDF)
Before this commit: robot ec616, 7 links, 6 joints
Links:
- added link gripper_1_link, mass 0.0229473565168191; collision mesh filename=meshes/gripper_1_link.STL; visual mesh filename=meshes/gripper_1_link.STL
- added link gripper_2_link, mass 0.0229473565168191; collision mesh filename=meshes/gripper_1_link.STL scale=1 -1 1; visual mesh filename=meshes/gripper_1_link.STL scale=1 -1 1
- added link gripper_centor_link, mass 0.05; collision mesh filename=meshes/gripper_centor_link.STL; visual mesh filename=meshes/gripper_centor_link.STL
Joints:
- added joint gripper_1_joint: type revolute, parent Link6, child gripper_1_link, origin xyz=0.02916 0.0005 0.0105 rpy=-1.5708 -1.5708 0, axis 0 0 1, limit lower=0 upper=0.7 effort=20 velocity=0.35
- added joint gripper_2_joint: type revolute, parent Link6, child gripper_2_link, origin xyz=-0.02916 0.0005 0.0105 rpy=-1.5708 -1.5708 0, axis 0 0 1, limit lower=-0.7 upper=0.7 effort=20 velocity=0.35
- added joint gripper_centor_fixed: type fixed, parent Link6, child gripper_centor_link, origin xyz=0 0 0.025 rpy=0 0 0
- joint Joint1: limit lower=0 upper=0 effort=0 velocity=0 -> lower=-4.188 upper=4.188 effort=100.0 velocity=0.35
- joint Joint2: limit lower=0 upper=0 effort=0 velocity=0 -> lower=-4.188 upper=2.094 effort=100.0 velocity=0.35
- joint Joint3: limit lower=0 upper=0 effort=0 velocity=0 -> lower=-4.188 upper=2.094 effort=100.0 velocity=0.35
- joint Joint4: limit lower=0 upper=0 effort=0 velocity=0 -> lower=-4.188 upper=2.094 effort=100.0 velocity=0.35
- joint Joint5: limit lower=0 upper=0 effort=0 velocity=0 -> lower=-4.188 upper=2.094 effort=100.0 velocity=0.35
- joint Joint6: limit lower=0 upper=0 effort=0 velocity=0 -> lower=-4.188 upper=2.094 effort=100.0 velocity=0.35
